File: board/eggfckr.brd (EAGLE design)
At the start: 53.6 x 21.6 mm, 8 parts, among them U1 ATTINY85-20PU

Commit message: added btn WIP
Connections:
- removed net N$4: S1.P$2, U1.1
- net GND: now also S1.P$1
- net N$5: now also S1.P$2; no longer S1.P$1
Changed lines of the file:
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@@
 <contactref element="GND" pad="1"/>
 <contactref element="LED1" pad="K"/>
+<contactref element="S1" pad="P$1"/>
+<wire x1="23.495" y1="5.715" x2="31.09" y2="17.78" width="0" layer="19" extent="1-1"/>
 <wire x1="26.035" y1="2.54" x2="23.495" y2="5.715" width="0" layer="19" extent="1-1"/>
 <wire x1="7.62" y1="5.715" x2="23.495" y2="5.715" width="0" layer="19" extent="1-1"/>
@@
 </signal>
 <signal name="N$5">
-<contactref element="S1" pad="P$1"/>
 <contactref element="U1" pad="2"/>
-<wire x1="23.495" y1="10.795" x2="31.09" y2="17.78" width="0" layer="19" extent="1-1"/>
+<contactref element="S1" pad="P$2"/>
+<wire x1="23.495" y1="10.795" x2="24.79" y2="17.78" width="0" layer="19" extent="1-1"/>
 </signal>
 <signal name="N$2">
@@
 <wire x1="23.495" y1="8.255" x2="20.32" y2="8.255" width="0" layer="19" extent="1-16"/>
 </signal>
-<signal name="N$4">
-<contactref element="U1" pad="1"/>
-<contactref element="S1" pad="P$2"/>
-<wire x1="23.495" y1="13.335" x2="24.79" y2="17.78" width="0" layer="19" extent="1-1"/>
-</signal>
 <signal name="N$3">
