File: board/eggfckr.sch (EAGLE design)
At the start: 8 parts, among them U1 ATTINY85-20PU

Commit message: flipped LEDon pin2
Changed lines of the file:
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@@
 <part name="LED2" library="adafruit" deviceset="LED" device="3MM"/>
 <part name="GND2" library="ATtami" deviceset="GND" device=""/>
-<part name="P+2" library="ATTiny Fuse Reset with 12V Charge Pump" deviceset="VCC" device=""/>
 <part name="GND1" library="ATtami" deviceset="GND" device=""/>
 <part name="P+3" library="ATTiny Fuse Reset with 12V Charge Pump" deviceset="VCC" device=""/>
@@
 </plain>
 <instances>
-<instance part="P+1" gate="VCC" x="78.74" y="27.94"/>
+<instance part="P+1" gate="VCC" x="78.74" y="30.48"/>
 <instance part="LED1" gate="G$1" x="2.54" y="22.86" rot="R90"/>
 <instance part="R2" gate="G$1" x="63.5" y="20.32" smashed="yes" rot="R180">
@@
 <instance part="LED2" gate="G$1" x="76.2" y="20.32" rot="R270"/>
 <instance part="GND2" gate="1" x="0" y="5.08"/>
-<instance part="P+2" gate="VCC" x="78.74" y="7.62" rot="R180"/>
 <instance part="GND1" gate="1" x="20.32" y="5.08"/>
 <instance part="P+3" gate="VCC" x="0" y="30.48"/>
@@
 <pinref part="R2" gate="G$1" pin="2"/>
 <wire x1="58.42" y1="20.32" x2="55.88" y2="20.32" width="0.1524" layer="91"/>
-</segment>
-</net>
-<net name="N$6" class="0">
-<segment>
-<pinref part="R1" gate="G$1" pin="1"/>
-<pinref part="LED1" gate="G$1" pin="C"/>
 </segment>
 </net>
@@
 <net name="VCC" class="0">
 <segment>
+<pinref part="LED2" gate="G$1" pin="A"/>
 <pinref part="P+1" gate="VCC" pin="VCC"/>
+<wire x1="78.74" y1="20.32" x2="78.74" y2="25.4" width="0.1524" layer="91"/>
 <pinref part="U1" gate="A" pin="(VCC)8"/>
+<wire x1="78.74" y1="25.4" x2="78.74" y2="27.94" width="0.1524" layer="91"/>
 <wire x1="55.88" y1="25.4" x2="78.74" y2="25.4" width="0.1524" layer="91"/>
-</segment>
-<segment>
-<pinref part="LED2" gate="G$1" pin="A"/>
-<pinref part="P+2" gate="VCC" pin="VCC"/>
-<wire x1="78.74" y1="20.32" x2="78.74" y2="10.16" width="0.1524" layer="91"/>
-</segment>
-<segment>
-<pinref part="LED1" gate="G$1" pin="A"/>
-<pinref part="P+3" gate="VCC" pin="VCC"/>
-<wire x1="0" y1="22.86" x2="0" y2="27.94" width="0.1524" layer="91"/>
-<wire x1="0" y1="22.86" x2="0" y2="17.78" width="0.1524" layer="91"/>
-<junction x="0" y="22.86"/>
-<pinref part="R3" gate="R" pin="3"/>
+<junction x="78.74" y="25.4"/>
 </segment>
 <segment>
@@
 <pinref part="VCC" gate="G$1" pin="1"/>
 <wire x1="48.26" y1="45.72" x2="48.26" y2="40.64" width="0.1524" layer="91"/>
+</segment>
+<segment>
+<pinref part="P+3" gate="VCC" pin="VCC"/>
+<pinref part="LED1" gate="G$1" pin="A"/>
+<wire x1="0" y1="27.94" x2="0" y2="22.86" width="0.1524" layer="91"/>
+<pinref part="R3" gate="R" pin="3"/>
+<wire x1="0" y1="22.86" x2="0" y2="17.78" width="0.1524" layer="91"/>
+<junction x="0" y="22.86"/>
 </segment>
 </net>
@@
 </segment>
 </net>
+<net name="N$3" class="0">
+<segment>
+<pinref part="R1" gate="G$1" pin="1"/>
+<pinref part="LED1" gate="G$1" pin="C"/>
+</segment>
+</net>

Commit message: changed routing
Parts:
- removed R3: (no value), dp_devices:TRIMMER-3306F
- added S1: SWITCH-MOMENTARY-2-SMD-1101NE, ATtami:SWITCH-MOMENTARY-2-SMD-1101NE
Connections:
- new net N$5: S1.1, U1.2(PB3)
- net GND: now also LED1.C; no longer R3.1
- net N$2: now also R1.2; no longer R3.2
- net N$3: now also LED1.A; no longer LED1.C
- net N$4: now also S1.2, U1.1(PB5); no longer R1.2, U1.2(PB3)
- net VCC: no longer LED1.A, R3.3
Other:
- moved on the sheet: GND, LED1, VCC
Changed lines of the file:
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@@
 <?xml version="1.0" encoding="utf-8"?>
 <!DOCTYPE eagle SYSTEM "eagle.dtd">
-<eagle version="7.2.0">
+<eagle version="7.1.0">
 <drawing>
 <settings>
@@
 <part name="R1" library="adafruit" deviceset="R-US_" device="0204/7"/>
 <part name="LED2" library="adafruit" deviceset="LED" device="3MM"/>
-<part name="GND2" library="ATtami" deviceset="GND" device=""/>
-<part name="GND1" library="ATtami" deviceset="GND" device=""/>
-<part name="P+3" library="ATTiny Fuse Reset with 12V Charge Pump" deviceset="VCC" device=""/>
 <part name="P+4" library="ATTiny Fuse Reset with 12V Charge Pump" deviceset="VCC" device=""/>
 <part name="GND3" library="ATtami" deviceset="GND" device=""/>
-<part name="R3" library="dp_devices" deviceset="TRIMMER" device="-3306F"/>
 <part name="GND" library="microbuilder" deviceset="HEADER-1X1" device="ROUND"/>
 <part name="VCC" library="microbuilder" deviceset="HEADER-1X1" device="ROUND"/>
+<part name="S1" library="ATtami" deviceset="SWITCH-MOMENTARY-2" device="-SMD-1101NE"/>
+<part name="GND2" library="ATtami" deviceset="GND" device=""/>
 </parts>
 <sheets>
@@
 <instances>
 <instance part="P+1" gate="VCC" x="78.74" y="30.48"/>
-<instance part="LED1" gate="G$1" x="2.54" y="22.86" rot="R90"/>
+<instance part="LED1" gate="G$1" x="2.54" y="15.24" rot="R270"/>
 <instance part="R2" gate="G$1" x="63.5" y="20.32" smashed="yes" rot="R180">
 <attribute name="NAME" x="60.452" y="22.1234" size="1.27" layer="95" rot="R180"/>
@@
 <attribute name="VALUE" x="25.4762" y="4.445" size="2.0828" layer="96" ratio="10" rot="SR0"/>
 </instance>
-<instance part="R1" gate="G$1" x="12.7" y="22.86" smashed="yes">
-<attribute name="NAME" x="15.748" y="21.0566" size="1.27" layer="95"/>
-<attribute name="VALUE" x="8.89" y="19.558" size="1.778" layer="96"/>
+<instance part="R1" gate="G$1" x="12.7" y="15.24" smashed="yes">
+<attribute name="VALUE" x="8.89" y="11.938" size="1.778" layer="96"/>
 </instance>
 <instance part="LED2" gate="G$1" x="76.2" y="20.32" rot="R270"/>
-<instance part="GND2" gate="1" x="0" y="5.08"/>
-<instance part="GND1" gate="1" x="20.32" y="5.08"/>
-<instance part="P+3" gate="VCC" x="0" y="30.48"/>
-<instance part="P+4" gate="VCC" x="48.26" y="38.1" rot="R180"/>
-<instance part="GND3" gate="1" x="58.42" y="38.1"/>
-<instance part="R3" gate="R" x="0" y="12.7" rot="R90"/>
-<instance part="GND" gate="G$1" x="60.96" y="45.72" smashed="yes">
-<attribute name="NAME" x="54.61" y="48.895" size="1.778" layer="95"/>
-<attribute name="VALUE" x="54.61" y="40.64" size="1.778" layer="96"/>
-</instance>
-<instance part="VCC" gate="G$1" x="50.8" y="45.72" smashed="yes">
-<attribute name="NAME" x="44.45" y="48.895" size="1.778" layer="95"/>
-<attribute name="VALUE" x="44.45" y="40.64" size="1.778" layer="96"/>
-</instance>
+<instance part="P+4" gate="VCC" x="33.02" y="-15.24" rot="R180"/>
+<instance part="GND3" gate="1" x="43.18" y="-15.24"/>
+<instance part="GND" gate="G$1" x="45.72" y="-7.62" smashed="yes">
+<attribute name="NAME" x="39.37" y="-4.445" size="1.778" layer="95"/>
+<attribute name="VALUE" x="39.37" y="-12.7" size="1.778" layer="96"/>
+</instance>
+<instance part="VCC" gate="G$1" x="35.56" y="-7.62" smashed="yes">
+<attribute name="NAME" x="29.21" y="-4.445" size="1.778" layer="95"/>
+<attribute name="VALUE" x="29.21" y="-12.7" size="1.778" layer="96"/>
+</instance>
+<instance part="S1" gate="G$1" x="12.7" y="25.4" smashed="yes">
+<attribute name="NAME" x="10.16" y="27.94" size="1.778" layer="95"/>
+</instance>
+<instance part="GND2" gate="1" x="-5.08" y="2.54"/>
 </instances>
 <busses>
@@
 <segment>
 <pinref part="U1" gate="A" pin="4(GND)"/>
-<wire x1="20.32" y1="10.16" x2="20.32" y2="7.62" width="0.1524" layer="91"/>
-<pinref part="GND1" gate="1" pin="GND"/>
-</segment>
-<segment>
-<pinref part="R3" gate="R" pin="1"/>
+<pinref part="LED1" gate="G$1" pin="C"/>
+<wire x1="-2.54" y1="15.24" x2="-5.08" y2="15.24" width="0.1524" layer="91"/>
 <pinref part="GND2" gate="1" pin="GND"/>
+<wire x1="-5.08" y1="15.24" x2="-5.08" y2="7.62" width="0.1524" layer="91"/>
+<wire x1="-5.08" y1="7.62" x2="-5.08" y2="5.08" width="0.1524" layer="91"/>
+<wire x1="20.32" y1="10.16" x2="-2.54" y2="10.16" width="0.1524" layer="91"/>
+<wire x1="-2.54" y1="10.16" x2="-5.08" y2="7.62" width="0.1524" layer="91"/>
+<junction x="-5.08" y="7.62"/>
 </segment>
 <segment>
 <pinref part="GND3" gate="1" pin="GND"/>
 <pinref part="GND" gate="G$1" pin="1"/>
-<wire x1="58.42" y1="45.72" x2="58.42" y2="40.64" width="0.1524" layer="91"/>
+<wire x1="43.18" y1="-7.62" x2="43.18" y2="-12.7" width="0.1524" layer="91"/>
 </segment>
 </net>
 <net name="VCC" class="0">
 <segment>
+<pinref part="P+4" gate="VCC" pin="VCC"/>
+<pinref part="VCC" gate="G$1" pin="1"/>
+<wire x1="33.02" y1="-7.62" x2="33.02" y2="-12.7" width="0.1524" layer="91"/>
+</segment>
+<segment>
+<pinref part="U1" gate="A" pin="(VCC)8"/>
 <pinref part="LED2" gate="G$1" pin="A"/>
 <pinref part="P+1" gate="VCC" pin="VCC"/>
-<wire x1="78.74" y1="20.32" x2="78.74" y2="25.4" width="0.1524" layer="91"/>
-<pinref part="U1" gate="A" pin="(VCC)8"/>
-<wire x1="78.74" y1="25.4" x2="78.74" y2="27.94" width="0.1524" layer="91"/>
-<wire x1="55.88" y1="25.4" x2="78.74" y2="25.4" width="0.1524" layer="91"/>
-<junction x="78.74" y="25.4"/>
-</segment>
-<segment>
-<pinref part="P+4" gate="VCC" pin="VCC"/>
-<pinref part="VCC" gate="G$1" pin="1"/>
-<wire x1="48.26" y1="45.72" x2="48.26" y2="40.64" width="0.1524" layer="91"/>
-</segment>
-<segment>
-<pinref part="P+3" gate="VCC" pin="VCC"/>
+<wire x1="78.74" y1="20.32" x2="78.74" y2="27.94" width="0.1524" layer="91"/>
+<wire x1="55.88" y1="25.4" x2="76.2" y2="25.4" width="0.1524" layer="91"/>
+<wire x1="76.2" y1="25.4" x2="78.74" y2="27.94" width="0.1524" layer="91"/>
+<junction x="78.74" y="27.94"/>
+</segment>
+</net>
+<net name="N$5" class="0">
+<segment>
+<pinref part="S1" gate="G$1" pin="1"/>
+<wire x1="7.62" y1="20.32" x2="7.62" y2="25.4" width="0.1524" layer="91"/>
+<pinref part="U1" gate="A" pin="2(PB3)"/>
+<wire x1="20.32" y1="20.32" x2="7.62" y2="20.32" width="0.1524" layer="91"/>
+</segment>
+</net>
+<net name="N$2" class="0">
+<segment>
+<pinref part="R1" gate="G$1" pin="2"/>
+<pinref part="U1" gate="A" pin="3(PB4)"/>
+<wire x1="17.78" y1="15.24" x2="20.32" y2="15.24" width="0.1524" layer="91"/>
+</segment>
+</net>
+<net name="N$4" class="0">
+<segment>
+<pinref part="U1" gate="A" pin="1(PB5)"/>
+<pinref part="S1" gate="G$1" pin="2"/>
+<wire x1="20.32" y1="25.4" x2="17.78" y2="25.4" width="0.1524" layer="91"/>
+</segment>
+</net>
+<net name="N$3" class="0">
+<segment>
+<pinref part="R1" gate="G$1" pin="1"/>
 <pinref part="LED1" gate="G$1" pin="A"/>
-<wire x1="0" y1="27.94" x2="0" y2="22.86" width="0.1524" layer="91"/>
-<pinref part="R3" gate="R" pin="3"/>
-<wire x1="0" y1="22.86" x2="0" y2="17.78" width="0.1524" layer="91"/>
-<junction x="0" y="22.86"/>
-</segment>
-</net>
-<net name="N$4" class="0">
-<segment>
-<pinref part="U1" gate="A" pin="2(PB3)"/>
-<pinref part="R1" gate="G$1" pin="2"/>
-<wire x1="20.32" y1="20.32" x2="17.78" y2="22.86" width="0.1524" layer="91"/>
-</segment>
-</net>
-<net name="N$2" class="0">
-<segment>
-<pinref part="U1" gate="A" pin="3(PB4)"/>
-<wire x1="20.32" y1="12.7" x2="20.32" y2="15.24" width="0.1524" layer="91"/>
-<pinref part="R3" gate="R" pin="2"/>
-<wire x1="5.08" y1="12.7" x2="20.32" y2="12.7" width="0.1524" layer="91"/>
-</segment>
-</net>
-<net name="N$3" class="0">
-<segment>
-<pinref part="R1" gate="G$1" pin="1"/>
-<pinref part="LED1" gate="G$1" pin="C"/>
-</segment>
-</net>
+<wire x1="7.62" y1="15.24" x2="5.08" y2="15.24" width="0.1524" layer="91"/>
+</segment>
+</net>

Commit message: added btn WIP
Connections:
- removed net N$4: S1.2, U1.1(PB5)
- net GND: now also S1.1
- net N$5: now also S1.2; no longer S1.1
Other:
- moved on the sheet: S1
Changed lines of the file:
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@@
 <attribute name="VALUE" x="29.21" y="-12.7" size="1.778" layer="96"/>
 </instance>
-<instance part="S1" gate="G$1" x="12.7" y="25.4" smashed="yes">
-<attribute name="NAME" x="10.16" y="27.94" size="1.778" layer="95"/>
+<instance part="S1" gate="G$1" x="2.54" y="20.32" smashed="yes">
+<attribute name="NAME" x="0" y="22.86" size="1.778" layer="95"/>
 </instance>
 <instance part="GND2" gate="1" x="-5.08" y="2.54"/>
@@
 <wire x1="-2.54" y1="10.16" x2="-5.08" y2="7.62" width="0.1524" layer="91"/>
 <junction x="-5.08" y="7.62"/>
+<wire x1="-5.08" y1="15.24" x2="-5.08" y2="17.78" width="0.1524" layer="91"/>
+<junction x="-5.08" y="15.24"/>
+<pinref part="S1" gate="G$1" pin="1"/>
+<wire x1="-5.08" y1="17.78" x2="-2.54" y2="20.32" width="0.1524" layer="91"/>
 </segment>
 <segment>
@@
 <net name="N$5" class="0">
 <segment>
-<pinref part="S1" gate="G$1" pin="1"/>
-<wire x1="7.62" y1="20.32" x2="7.62" y2="25.4" width="0.1524" layer="91"/>
 <pinref part="U1" gate="A" pin="2(PB3)"/>
 <wire x1="20.32" y1="20.32" x2="7.62" y2="20.32" width="0.1524" layer="91"/>
+<pinref part="S1" gate="G$1" pin="2"/>
 </segment>
 </net>
@@
 </segment>
 </net>
-<net name="N$4" class="0">
-<segment>
-<pinref part="U1" gate="A" pin="1(PB5)"/>
-<pinref part="S1" gate="G$1" pin="2"/>
-<wire x1="20.32" y1="25.4" x2="17.78" y2="25.4" width="0.1524" layer="91"/>
-</segment>
-</net>
