File: board/eggfckr.sch (EAGLE design)
At the start: 8 parts, among them U1 ATTINY85-20PU

Commit message: whats going on'
Parts:
- removed GND, VCC: (no value), microbuilder:HEADER-1X1ROUND
- removed R1, R2: (no value), adafruit:R-US_0204/7
- removed S1: SWITCH-MOMENTARY-2-SMD-1101NE, ATtami:SWITCH-MOMENTARY-2-SMD-1101NE
- removed U1: ATTINY85-20PU, Atmel_By_element14_Batch_1-00:ATTINY85-20PU
- added +, -: (no value), eggfckr:HEADER-1X1
- added ATINY85: ATTINY85-20PU, eggfckr:ATTINY85-20PU
- added R3: (no value), eggfckr:TRIMMER-3306F
Connections:
- removed net N$4: S1.2, U1.1(PB5)
- removed net N$5: S1.1, U1.2(PB3)
- removed net N$7: LED2.C, R2.1
- net GND: now also -.1, ATINY85.4(GND), R3.1; no longer GND.1, LED1.C, U1.4(GND)
- net N$1: now also ATINY85.(PB2)7, LED2.A; no longer R2.2, U1.(PB2)7
- net N$2: now also ATINY85.3(PB4), R3.2; no longer R1.2, U1.3(PB4)
- net N$3: now also ATINY85.2(PB3), LED1.C; no longer LED1.A, R1.1
- net VCC: now also +.1, ATINY85.(VCC)8, LED1.A, LED2.C, R3.3; no longer LED2.A, U1.(VCC)8, VCC.1
Other:
- note removed: "eegfckr"
- moved on the sheet: LED1, LED2
